File: TP2/pcb-instrumento-virtual/instrumento_virtual/_autosave-instrumento_virtual.kicad_pcb (KiCad board)
At the start: 2 copper layers, 90 parts, among them J1 Conn_01x09_Pin, J2 Conector_salidas_analógicas, J3 Conn_01x20_Socket, J4 Conn_01x09_Pin, J5 Conn_01x20_Socket, J7 RS232, Q10 BC547, Q3 BC547, Q4 BC547, Q5 BC547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

Commit message: primera versión tentativa de esquemático
Parts:
- U2, U6: footprint Package_DFN_QFN:DFN-8-1EP_3x2mm_P0.5mm_EP1.75x1.45mm -> Package_DIP:DIP-8_W7.62mm
- moved J1 171.9 mm to (223.5, 127.0), turned to 180 degrees
- moved C15 167.0 mm to (213.4, 83.8), turned to 90 degrees
- moved U5 133.9 mm to (203.2, 83.8), turned to 90 degrees
- moved D2 130.0 mm to (175.3, 123.2), turned to -90 degrees
- moved R45 127.8 mm to (137.0, 126.1), turned to 90 degrees
- moved R43 127.2 mm to (137.0, 117.1), turned to 90 degrees
- moved U4 126.8 mm to (190.7, 83.8), turned to 90 degrees
- moved R41 126.7 mm to (137.0, 108.1), turned to 90 degrees
- moved D1 125.7 mm to (175.3, 113.0), turned to -90 degrees
- moved R40 123.0 mm to (137.0, 98.5), turned to 90 degrees
- moved R31 118.0 mm to (123.0, 111.9), turned to -90 degrees
- moved R46 117.9 mm to (127.0, 126.1), turned to 90 degrees
- moved R44 117.2 mm to (127.0, 117.0), turned to 90 degrees
- moved C18 114.9 mm to (180.3, 83.8), turned to -90 degrees
- moved C5 114.7 mm to (40.6, 147.3), turned to -90 degrees
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Routing:
- net 3.3V: track 0.00 -> 82.6 mm, vias 0 -> 2
- net 5V: track 0.00 -> 71.3 mm
- net PB15: track 0.00 -> 64.9 mm
- net PB3: track 0.00 -> 63.2 mm
- net DOUT8: track 0.00 -> 60.2 mm
- net PA10: track 0.00 -> 44.6 mm
- net DOUT3: track 0.00 -> 24.5 mm
- net PA9: track 0.00 -> 22.4 mm
- net PB5: track 0.00 -> 20.9 mm
- net PB4: track 0.00 -> 18.6 mm
- net PA8: track 0.00 -> 17.9 mm
- net DOUT6: track 0.00 -> 9.38 mm
- net DOUT2: track 0.00 -> 8.38 mm
- net Net-(Q4-B): track 0.00 -> 8.26 mm
- net Net-(Q7-B): track 0.00 -> 7.61 mm
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